File: miura_board.kicad_sch (KiCad schematic)
At the start: 22 parts, among them J1 Conn_01x02_Female, SW1 SW_Push, U1 ATmega32U4-A, U2 NRF24L01, Y1 16MHz, Y2 16MHz

Commit message: Square
Parts:
- added J2, J3: Screw_Terminal_01x02, TerminalBlock_Phoenix:TerminalBlock_Phoenix_MPT-0,5-2-2.54_1x02_P2.54mm_Horizontal, symbol Connector:Screw_Terminal_01x02
- added U3, U4: DRV8833PW, Package_SO:TSSOP-16_4.4x5mm_P0.65mm, symbol Driver_Motor:DRV8833PW
Changed lines of the file:
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@@
     (pin "9")
+  )
+  (symbol (lib_id "Connector:Screw_Terminal_01x02") (at 245.11 39.37 0) (unit 1)
+    (in_bom yes) (on_board yes) (fields_autoplaced)
+    (property "Reference" "J3" (id 0) (at 247.142 39.8053 0)
+      (effects (font (size 1.27 1.27)) (justify left))
+    )
+    (property "Value" "Screw_Terminal_01x02" (id 1) (at 247.142 42.3422 0)
+      (effects (font (size 1.27 1.27)) (justify left))
+    )
+    (property "Footprint" "TerminalBlock_Phoenix:TerminalBlock_Phoenix_MPT-0,5-2-2.54_1x02_P2.54mm_Horizontal" (id 2) (at 245.11 39.37 0)
+      (effects (font (size 1.27 1.27)) hide)
+    )
+    (property "Datasheet" "~" (id 3) (at 245.11 39.37 0)
+      (effects (font (size 1.27 1.27)) hide)
+    )
+    (pin "1")
+    (pin "2")
   )
   (symbol (lib_id "power:GND") (at 73.66 95.25 0) (unit 1)
@@
     (pin "2")
   )
+  (symbol (lib_id "Driver_Motor:DRV8833PW") (at 214.63 73.66 0) (unit 1)
+    (in_bom yes) (on_board yes) (fields_autoplaced)
+    (property "Reference" "U3" (id 0) (at 216.6494 88.3904 0)
+      (effects (font (size 1.27 1.27)) (justify left))
+    )
+    (property "Value" "DRV8833PW" (id 1) (at 216.6494 90.9273 0)
+      (effects (font (size 1.27 1.27)) (justify left))
+    )
+    (property "Footprint" "Package_SO:TSSOP-16_4.4x5mm_P0.65mm" (id 2) (at 226.06 62.23 0)
+      (effects (font (size 1.27 1.27)) (justify left) hide)
+    )
+    (property "Datasheet" "http://www.ti.com/lit/ds/symlink/drv8833.pdf" (id 3) (at 210.82 59.69 0)
+      (effects (font (size 1.27 1.27)) hide)
+    )
+    (pin "1")
+    (pin "10")
+    (pin "11")
+    (pin "12")
+    (pin "13")
+    (pin "14")
+    (pin "15")
+    (pin "16")
+    (pin "2")
+    (pin "3")
+    (pin "4")
+    (pin "5")
+    (pin "6")
+    (pin "7")
+    (pin "8")
+    (pin "9")
+  )
   (symbol (lib_id "Device:R_Small") (at 110.49 110.49 90) (unit 1)
     (in_bom yes) (on_board yes)
@@
     (pin "1")
     (pin "2")
+  )
+  (symbol (lib_id "Driver_Motor:DRV8833PW") (at 257.81 73.66 0) (unit 1)
+    (in_bom yes) (on_board yes) (fields_autoplaced)
+    (property "Reference" "U4" (id 0) (at 259.8294 88.3904 0)
+      (effects (font (size 1.27 1.27)) (justify left))
+    )
+    (property "Value" "DRV8833PW" (id 1) (at 259.8294 90.9273 0)
+      (effects (font (size 1.27 1.27)) (justify left))
+    )
+    (property "Footprint" "Package_SO:TSSOP-16_4.4x5mm_P0.65mm" (id 2) (at 269.24 62.23 0)
+      (effects (font (size 1.27 1.27)) (justify left) hide)
+    )
+    (property "Datasheet" "http://www.ti.com/lit/ds/symlink/drv8833.pdf" (id 3) (at 254 59.69 0)
+      (effects (font (size 1.27 1.27)) hide)
+    )
+    (pin "1")
+    (pin "10")
+    (pin "11")
+    (pin "12")
+    (pin "13")
+    (pin "14")
+    (pin "15")
+    (pin "16")
+    (pin "2")
+    (pin "3")
+    (pin "4")
+    (pin "5")
+    (pin "6")
+    (pin "7")
+    (pin "8")
+    (pin "9")
   )
   (symbol (lib_id "Device:Crystal_GND3") (at 123.19 54.61 0) (unit 1)
@@
     (pin "9")
   )
+  (symbol (lib_id "Connector:Screw_Terminal_01x02") (at 245.11 26.67 0) (unit 1)
+    (in_bom yes) (on_board yes) (fields_autoplaced)
+    (property "Reference" "J2" (id 0) (at 247.142 27.1053 0)
+      (effects (font (size 1.27 1.27)) (justify left))
+    )
+    (property "Value" "Screw_Terminal_01x02" (id 1) (at 247.142 29.6422 0)
+      (effects (font (size 1.27 1.27)) (justify left))
+    )
+    (property "Footprint" "TerminalBlock_Phoenix:TerminalBlock_Phoenix_MPT-0,5-2-2.54_1x02_P2.54mm_Horizontal" (id 2) (at 245.11 26.67 0)
+      (effects (font (size 1.27 1.27)) hide)
+    )
+    (property "Datasheet" "~" (id 3) (at 245.11 26.67 0)
+      (effects (font (size 1.27 1.27)) hide)
+    )
+    (pin "1")
+    (pin "2")
+  )
   (symbol (lib_id "Device:R_Small") (at 110.49 95.25 90) (unit 1)
     (in_bom yes) (on_board yes)
@@
       (reference "J1") (unit 1) (value "Conn_01x02_Female") (footprint "Connector_PinHeader_2.54mm:PinHeader_1x02_P2.54mm_Vertical")
     )
+    (path "/a84b7f14-d4af-4368-9497-c56d01da868d"
+      (reference "J2") (unit 1) (value "Screw_Terminal_01x02") (footprint "TerminalBlock_Phoenix:TerminalBlock_Phoenix_MPT-0,5-2-2.54_1x02_P2.54mm_Horizontal")
+    )
+    (path "/4df0df01-e01e-45d8-bf75-0c04b089b3fa"
+      (reference "J3") (unit 1) (value "Screw_Terminal_01x02") (footprint "TerminalBlock_Phoenix:TerminalBlock_Phoenix_MPT-0,5-2-2.54_1x02_P2.54mm_Horizontal")
+    )
     (path "/4719b1c6-0945-4abe-b9e1-a28e585215e5"
       (reference "R1") (unit 1) (value "22") (footprint "Resistor_SMD:R_0603_1608Metric_Pad0.98x0.95mm_HandSolder")
@@
       (reference "U2") (unit 1) (value "NRF24L01") (footprint "Package_DFN_QFN:QFN-20-1EP_4x4mm_P0.5mm_EP2.5x2.5mm")
     )
+    (path "/723fb764-14ee-4461-b800-e4d673c3e301"
+      (reference "U3") (unit 1) (value "DRV8833PW") (footprint "Package_SO:TSSOP-16_4.4x5mm_P0.65mm")
+    )
+    (path "/95d7d7ea-217d-4e85-bfe1-71e575081e16"
+      (reference "U4") (unit 1) (value "DRV8833PW") (footprint "Package_SO:TSSOP-16_4.4x5mm_P0.65mm")
+    )
     (path "/49d3b3eb-e418-4a5d-8c98-9ed478100523"

Commit message: Square
Parts:
- removed C1: 10uF, Capacitor_SMD:C_0603_1608Metric, symbol Device:C_Small
- removed R3: 10k, Resistor_SMD:R_0603_1608Metric_Pad0.98x0.95mm_HandSolder, symbol Device:R_Small
- removed U1: ATmega32U4-A, Package_QFP:TQFP-44_10x10mm_P0.8mm, symbol MCU_Microchip_ATmega:ATmega32U4-A
- added U5: ESP32-S2-SOLO, Espressif:ESP32-S2-SOLO, symbol Espressif:ESP32-S2-SOLO
Connections:
- net GND: now also U5.1 (GND), U5.40 (GND), U5.41 (GND)
- net at R2.1: now also U5.13 (GPIO19/U1RTS/ADC2_CH8/CLK_OUT2/USB_D-)
- net at R1.2: now also U5.14 (GPIO20/U1CTS/ADC2_CH9/CLK_OUT1/USB_D+)
Other:
- moved on the sheet: D1, J1, R1, R2, R5, R6, R7, USB1

Commit message: Added ESP32
Parts:
- removed C4, C7: 0.1uF, Capacitor_SMD:C_0603_1608Metric, symbol Device:C_Small
- removed U2: NRF24L01, Package_DFN_QFN:QFN-20-1EP_4x4mm_P0.5mm_EP2.5x2.5mm, symbol RF:NRF24L01
- removed U5: ESP32-S2-SOLO, Espressif:ESP32-S2-SOLO, symbol Espressif:ESP32-S2-SOLO
- removed Y1, Y2: 16MHz, Crystal:Resonator-3Pin_W7.0mm_H2.5mm, symbol Device:Crystal_GND3
- added C? (x4): 10uF, Capacitor_SMD:C_0603_1608Metric, symbol Device:C_Small
- added C? (x6): 0.1uF, Capacitor_SMD:C_0603_1608Metric, symbol Device:C_Small
- added H? (x4): MountingHole_Pad, symbol Mechanical:MountingHole_Pad
- added R?: 22k, Resistor_SMD:R_0603_1608Metric_Pad0.98x0.95mm_HandSolder, symbol Device:R_Small
- added R?: 47k, Resistor_SMD:R_0603_1608Metric_Pad0.98x0.95mm_HandSolder, symbol Device:R_Small
- added U1: ESP32-WROOM, ESP32-footprints-Lib:ESP32-WROOM, symbol ESP32-footprints-Shem-Lib:ESP32-WROOM
- added U?: AMS1117, Package_TO_SOT_SMD:SOT-223-3_TabPin2, symbol Regulator_Linear:AMS1117
- added U?: CP2102N-Axx-xQFN24, Package_DFN_QFN:QFN-24-1EP_4x4mm_P0.5mm_EP2.6x2.6mm, symbol Interface_USB:CP2102N-Axx-xQFN24
Connections:
- net +5V: now also C?.1, C?.1, R?.1, U?.3 (VI); no longer D1.2 (A), R4.1
- net GND: now also C?.2, C?.2, C?.2, C?.2, C?.2, C?.2, C?.2, C?.2, C?.2, C?.2, H?.1, H?.1, H?.1, H?.1, R?.1, U?.1 (ADJ), U?.2 (GND), U?.25 (GND)
- net at R1.2: now also U?.3 (D+)
- net at R2.1: now also U?.4 (D-)
- new net: R?.2, R?.2, U?.8 (VBUS)
- new net +3V3: C?.1, C?.1, C?.1, C?.1, C?.1, C?.1, C?.1, C?.1, D1.2 (A), U1.2 (3V3), U1.3 (EN), U?.2 (VO), U?.5 (VIO), U?.6 (VDD), U?.7 (VREGIN)
- new net RXD: U1.34 (RXD0), U?.20 (RXD)
- new net TXD: U1.35 (TXD0), U?.21 (TXD)
Other:
- moved on the sheet: R1, R2

Commit message: STEP
Parts:
- removed C? (x2): 0.1uF, Capacitor_SMD:C_0603_1608Metric, symbol Device:C_Small
- removed R2: 22, Resistor_SMD:R_0603_1608Metric_Pad0.98x0.95mm_HandSolder, symbol Device:R_Small
- removed R4: 10k, Resistor_SMD:R_0603_1608Metric_Pad0.98x0.95mm_HandSolder, symbol Device:R_Small
- removed R?: 22k, Resistor_SMD:R_0603_1608Metric_Pad0.98x0.95mm_HandSolder, symbol Device:R_Small
- removed R?: 47k, Resistor_SMD:R_0603_1608Metric_Pad0.98x0.95mm_HandSolder, symbol Device:R_Small
- removed U?: CP2102N-Axx-xQFN24, Package_DFN_QFN:QFN-24-1EP_4x4mm_P0.5mm_EP2.6x2.6mm, symbol Interface_USB:CP2102N-Axx-xQFN24
- added C14, C15, C16, C7: 0.1uF, Capacitor_SMD:C_0603_1608Metric, symbol Device:C_Small
- added J4: Conn_01x04_Male, Connector_PinHeader_2.54mm:PinHeader_1x04_P2.54mm_Vertical, symbol Connector:Conn_01x04_Male
- added J5, J6, J7: Screw_Terminal_01x02, TerminalBlock_Phoenix:TerminalBlock_Phoenix_MPT-0,5-2-2.54_1x02_P2.54mm_Horizontal, symbol Connector:Screw_Terminal_01x02
- added SW2: SW_Push, Button_Switch_THT:SW_PUSH-12mm, symbol Switch:SW_Push
- added U2: W25Q32JVSS, Package_SO:SOIC-8_5.23x5.23mm_P1.27mm, symbol Memory_Flash:W25Q32JVSS
- added U6: MPU-6050, Sensor_Motion:InvenSense_QFN-24_4x4mm_P0.5mm, symbol Sensor_Motion:MPU-6050
- H1, H2, H3, H4: renamed from H?; footprint (none) -> MountingHole:MountingHole_2.2mm_M2_DIN965_Pad
- R1: value 22 -> 10k
- gave numbers to parts that had none: 9
Connections:
- net RESET is gone; now on net GND: SW1.2
- net +3V3: now also R1.1, C15.1, U2.8 (VCC), U6.13 (VDD), U6.8 (VDDIO); no longer U1.3 (EN)
- net D+: no longer R1.1
- net GND: now also U1.1 (GND), U1.15 (GND), U1.38 (GND), U1.39 (GND-PAD), C14.1, C14.2, C15.2, C16.2, C7.1, C7.2, J4.3 (Pin_3), J5.2 (Pin_2), SW2.2, U2.4 (GND), U6.11 (FSYNC), U6.18 (GND), U6.20 (CPOUT); no longer SW1.1
- net at R1.2: now also SW1.1, U1.3 (EN)
- net at J3.1 (Pin_1): now also U4.2 (AOUT1)
- net at J3.2 (Pin_2): now also U4.4 (AOUT2)
- net MOTOR_B12_IN: now reaches U1.10 (IO25)
- net MOTOR_B12_IN: now also U3.10 (BIN2)
- net MOTOR_B11_IN: now reaches U1.11 (IO26)
- net MOTOR_B11_IN: now also U3.9 (BIN1)
- net MOTOR_A12_IN: now reaches U1.12 (IO27)
- net MOTOR_A12_IN: now also U3.15 (AIN2)
- net MOTOR_A11_IN: now reaches U1.13 (IO14)
- net MOTOR_A11_IN: now also U3.16 (AIN1)
- net SPI_CS: now reaches U1.19 (CMD)
- net SPI_CS: now also U2.1 (~{CS})
- net SPI_CLK: now reaches U1.20 (CLK)
- net SPI_CLK: now also U2.6 (CLK)
- net MISO: now reaches U1.21 (SDO)
- net MISO: now also U2.2 (DO(IO1))
- net MOSI: now reaches U1.22 (SD1)
- net MOSI: now also U2.5 (DI(IO0))
- net at U1.25 (IO0): now also SW2.1
- net SDA: now reaches U1.33 (IO21)
- net SDA: now also U6.24 (SDA)
- net SCL: now reaches U1.36 (IO22)
- net SCL: now also U6.23 (SCL)
- net MOTOR_B22_IN: now reaches U1.6 (IO34)
- net MOTOR_B22_IN: now also U4.10 (BIN2)
- net MOTOR_B21_IN: now reaches U1.7 (IO35)
- net MOTOR_B21_IN: now also U4.9 (BIN1)
- net MOTOR_A22_IN: now reaches U1.8 (IO32)
- net MOTOR_A22_IN: now also U4.15 (AIN2)
- net MOTOR_A21_IN: now reaches U1.9 (IO33)
- net MOTOR_A21_IN: now also U4.16 (AIN1)
- net MOTOR_SUPPLY: now reaches U3.12 (VM)
- net MOTOR_SUPPLY: now also U4.12 (VM), J5.1 (Pin_1)
- net at U3.2 (AOUT1): now also J6.1 (Pin_1)
- net at U3.4 (AOUT2): now also J6.2 (Pin_2)
- net at U3.5 (BOUT2): now also J2.2 (Pin_2)
- net at U3.7 (BOUT1): now also J2.1 (Pin_1)
- net at U4.5 (BOUT2): now also J7.2 (Pin_2)
- net at U4.7 (BOUT1): now also J7.1 (Pin_1)
- net RXD renamed RXD0
- net RXD0: now also J4.2 (Pin_2)
- net TXD renamed TXD0
- net TXD0: now also J4.1 (Pin_1)
- new net: C16.1, U6.10 (REGOUT)
Other:
- note added: "BOOT"
- note added: "Notes: - Move battery charging off board - Stretch would be wirless - Minimum would be microcontroller and motor contoller - 3.3 Operating voltage - SPI Flash for high memory kalmaan potential."
- note added: "RESET"
- note removed: "Notes: - Move battery charging off board - Stretch would be wirless - Minimum would be microcontroller and motor contoller - 2.4 - 5.0V Operating Voltage"
- moved on the sheet: C10, C11, C12, C13, J2, J3, U1, U3, U4
