File: _autosave-miura_board.kicad_sch (KiCad schematic)
At the start: 47 parts, among them J1 Screw_Terminal_01x02, J2 Screw_Terminal_01x02, J3 Screw_Terminal_01x02, J4 Conn_01x04_Male, J5 Screw_Terminal_01x02, J6 Screw_Terminal_01x02, J7 Screw_Terminal_01x02, J8 Screw_Terminal_01x02, SW1 SW_Push, SW2 SW_Push, U1 ESP32-WROOM, U3 DRV8833PW, U4 DRV8833PW, U5 AMS1117, U6 MPU-6050, U7 L7806, U8 DRV8833PW

Commit message: Add bypass
Parts:
- gave numbers to parts that had none: 3
Changed lines of the file:
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@@
   (symbol (lib_id "Device:C_Small") (at 64.77 68.58 0) (unit 1)
     (in_bom yes) (on_board yes) (fields_autoplaced)
-    (property "Reference" "C?" (id 0) (at 67.0941 67.7516 0)
+    (property "Reference" "C23" (id 0) (at 67.0941 67.7516 0)
       (effects (font (size 1.27 1.27)) (justify left))
     )
@@
   (symbol (lib_id "power:GND") (at 64.77 71.12 0) (unit 1)
     (in_bom yes) (on_board yes) (fields_autoplaced)
-    (property "Reference" "#PWR?" (id 0) (at 64.77 77.47 0)
+    (property "Reference" "#PWR0104" (id 0) (at 64.77 77.47 0)
       (effects (font (size 1.27 1.27)) hide)
     )
@@
   (symbol (lib_id "power:GND") (at 147.32 71.12 0) (unit 1)
     (in_bom yes) (on_board yes)
-    (property "Reference" "#PWR?" (id 0) (at 147.32 77.47 0)
+    (property "Reference" "#PWR0116" (id 0) (at 147.32 77.47 0)
       (effects (font (size 1.27 1.27)) hide)
     )
@@
   (symbol (lib_id "power:GND") (at 218.44 114.3 0) (unit 1)
     (in_bom yes) (on_board yes)
-    (property "Reference" "#PWR?" (id 0) (at 218.44 120.65 0)
+    (property "Reference" "#PWR0139" (id 0) (at 218.44 120.65 0)
       (effects (font (size 1.27 1.27)) hide)
     )
@@
   (symbol (lib_id "Device:C_Small") (at 147.32 68.58 0) (unit 1)
     (in_bom yes) (on_board yes) (fields_autoplaced)
-    (property "Reference" "C?" (id 0) (at 149.6441 67.7516 0)
+    (property "Reference" "C24" (id 0) (at 149.6441 67.7516 0)
       (effects (font (size 1.27 1.27)) (justify left))
     )
@@
   (symbol (lib_id "Device:C_Small") (at 218.44 111.76 0) (unit 1)
     (in_bom yes) (on_board yes) (fields_autoplaced)
-    (property "Reference" "C?" (id 0) (at 220.7641 110.9316 0)
+    (property "Reference" "C25" (id 0) (at 220.7641 110.9316 0)
       (effects (font (size 1.27 1.27)) (justify left))
     )
@@
       (reference "#PWR0103") (unit 1) (value "GND") (footprint "")
     )
+    (path "/07c002a7-300c-41aa-86e6-8fcffd0c0abf"
+      (reference "#PWR0104") (unit 1) (value "GND") (footprint "")
+    )
     (path "/9e8915db-19e2-42b4-9012-992ec98db144"
       (reference "#PWR0105") (unit 1) (value "GND") (footprint "")
@@
       (reference "#PWR0115") (unit 1) (value "GND") (footprint "")
     )
+    (path "/11a0282c-2364-4c90-8834-ccce88592545"
+      (reference "#PWR0116") (unit 1) (value "GND") (footprint "")
+    )
     (path "/61636e75-d6ce-474f-991e-bfd345f542d1"
       (reference "#PWR0117") (unit 1) (value "GND") (footprint "")
@@
       (reference "#PWR0138") (unit 1) (value "GND") (footprint "")
     )
-    (path "/07c002a7-300c-41aa-86e6-8fcffd0c0abf"
-      (reference "#PWR?") (unit 1) (value "GND") (footprint "")
-    )
-    (path "/11a0282c-2364-4c90-8834-ccce88592545"
-      (reference "#PWR?") (unit 1) (value "GND") (footprint "")
-    )
     (path "/18f9d82c-12a9-4f9a-ae4b-e6e3cce71393"
-      (reference "#PWR?") (unit 1) (value "GND") (footprint "")
+      (reference "#PWR0139") (unit 1) (value "GND") (footprint "")
     )
     (path "/4c630831-a484-4458-868e-601cdf4c800b"
@@
     )
     (path "/018c1408-69a7-4438-8025-b18adb265847"
-      (reference "C?") (unit 1) (value "10uF") (footprint "Capacitor_SMD:C_0603_1608Metric")
+      (reference "C23") (unit 1) (value "10uF") (footprint "Capacitor_SMD:C_0603_1608Metric")
     )
     (path "/6e286bc1-43b6-456b-b3a5-af6e83f0e01a"
-      (reference "C?") (unit 1) (value "10uF") (footprint "Capacitor_SMD:C_0603_1608Metric")
+      (reference "C24") (unit 1) (value "10uF") (footprint "Capacitor_SMD:C_0603_1608Metric")
     )
     (path "/cd5c2df4-e9ce-437e-adfa-53e9452b5bd9"
-      (reference "C?") (unit 1) (value "10uF") (footprint "Capacitor_SMD:C_0603_1608Metric")
+      (reference "C25") (unit 1) (value "10uF") (footprint "Capacitor_SMD:C_0603_1608Metric")
     )
     (path "/773333eb-e560-4953-905f-ee8d319272b9"

Commit message: new version
Other:
- note added: "Notes: - Move battery charging off board - Minimum would be microcontroller and motor contoller - 3.3 Operating voltage - SPI Flash for high memory kalmaan potential. - Encoder circuit. - The regulator footprint is not right. - Get rid of screw terminal."
- note removed: "Notes: - Move battery charging off board - Minimum would be microcontroller and motor contoller - 3.3 Operating voltage - SPI Flash for high memory kalmaan potential."
Changed lines of the file:
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@@
     (stroke (width 0) (type default) (color 0 0 0 0))
   )
-  (text "Notes: \n - Move battery charging off board\n - Minimum would be microcontroller and motor contoller\n - 3.3 Operating voltage\n - SPI Flash for high memory kalmaan potential. \n\n"
-    (at 13.97 29.21 0)
+  (text "Notes: \n - Move battery charging off board\n - Minimum would be microcontroller and motor contoller\n - 3.3 Operating voltage\n - SPI Flash for high memory kalmaan potential.\n - Encoder circuit. \n - The regulator footprint is not right. \n - Get rid of screw terminal.\n\n"
+    (at 13.97 30.48 0)
     (effects (font (size 1.27 1.27)) (justify left bottom))
   )
