File: _autosave-miura_board.kicad_sch (KiCad schematic)
At the start: 47 parts, among them J1 Screw_Terminal_01x02, J2 Screw_Terminal_01x02, J3 Screw_Terminal_01x02, J4 Conn_01x04_Male, J5 Screw_Terminal_01x02, J6 Screw_Terminal_01x02, J7 Screw_Terminal_01x02, J8 Screw_Terminal_01x02, SW1 SW_Push, SW2 SW_Push, U1 ESP32-WROOM, U3 DRV8833PW, U4 DRV8833PW, U5 AMS1117, U6 MPU-6050, U7 L7806, U8 DRV8833PW

Commit message: four layer
Other:
- note added: "Notes: - Move battery charging off board - Minimum would be microcontroller and motor contoller - 3.3 Operating voltage - SPI Flash for high memory kalmaan potential. - Encoder circuit. - The regulator footprint is not right. - Get rid of screw terminal."
- note removed: "Notes: - Move battery charging off board - Minimum would be microcontroller and motor contoller - 3.3 Operating voltage - SPI Flash for high memory kalmaan potential."
Changed lines of the file:
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@@
     (stroke (width 0) (type default) (color 0 0 0 0))
   )
-  (text "Notes: \n - Move battery charging off board\n - Minimum would be microcontroller and motor contoller\n - 3.3 Operating voltage\n - SPI Flash for high memory kalmaan potential. \n\n"
-    (at 13.97 29.21 0)
+  (text "Notes: \n - Move battery charging off board\n - Minimum would be microcontroller and motor contoller\n - 3.3 Operating voltage\n - SPI Flash for high memory kalmaan potential.\n - Encoder circuit. \n - The regulator footprint is not right. \n - Get rid of screw terminal.\n\n"
+    (at 13.97 30.48 0)
     (effects (font (size 1.27 1.27)) (justify left bottom))
   )
