File: miura_board/_autosave-miura_board.kicad_pcb (KiCad board)
At the start: 4 copper layers, 55.9 x 52.4 mm, 40 parts, among them J1 Micro_SD_Card_Det, J2 Conn_01x04_Male, J4 Conn_01x04_Male, J6 Conn_01x02_Male, SW1 SW_Push, SW2 SW_Push, U1 ESP32-WROOM, U2 AMS1117, U3 CP2102N-Axx-xQFN28, U4 MCP73832-5-OT, U5 AMS1117, U6 MPU-6050

Commit message: Rehaul
Parts:
- C17: moved to B.Cu
- moved C17 70.8 mm to (78.3, 58.7), turned to 180 degrees
Changed lines of the file:
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@@
-    )
-  )
-  (footprint "Capacitor_SMD:C_0603_1608Metric" (layer "F.Cu")
-    (at 149.09 59.24)
-    (descr "Capacitor SMD 0603 (1608 Metric), square (rectangular) end terminal, IPC_7351 nominal, (Body size source: IPC-SM-782 page 76, https://www.pcb-3d.com/wordpress/wp-content/uploads/ipc-sm-782a_amendment_1_and_2.pdf), generated with kicad-footprint-generator")
-    (tags "capacitor")
-    (property "Sheetfile" "miura_board.kicad_sch")
-    (property "Sheetname" "")
-    (attr smd)
-    (fp_text reference "C17" (at 0 -1.43) (layer "F.SilkS")
-      (effects (font (size 1 1) (thickness 0.15)))
-    )
-    (fp_text value "0.1uF" (at 0 1.43) (layer "F.Fab")
-      (effects (font (size 1 1) (thickness 0.15)))
-    )
-    (fp_text user "${REFERENCE}" (at 0 0) (layer "F.Fab")
-      (effects (font (size 0.4 0.4) (thickness 0.06)))
-    )
-    (fp_line (start -0.14058 -0.51) (end 0.14058 -0.51) (layer "F.SilkS") (width 0.12))
-    (fp_line (start -0.14058 0.51) (end 0.14058 0.51) (layer "F.SilkS") (width 0.12))
-    (fp_line (start 1.48 0.73) (end -1.48 0.73) (layer "F.CrtYd") (width 0.05))
-    (fp_line (start -1.48 -0.73) (end 1.48 -0.73) (layer "F.CrtYd") (width 0.05))
-    (fp_line (start 1.48 -0.73) (end 1.48 0.73) (layer "F.CrtYd") (width 0.05))
-    (fp_line (start -1.48 0.73) (end -1.48 -0.73) (layer "F.CrtYd") (width 0.05))
-    (fp_line (start -0.8 0.4) (end -0.8 -0.4) (layer "F.Fab") (width 0.1))
-    (fp_line (start 0.8 -0.4) (end 0.8 0.4) (layer "F.Fab") (width 0.1))
-    (fp_line (start -0.8 -0.4) (end 0.8 -0.4) (layer "F.Fab") (width 0.1))
-    (fp_line (start 0.8 0.4) (end -0.8 0.4) (layer "F.Fab") (width 0.1))
-    (pad "1" smd roundrect (at -0.775 0) (size 0.9 0.95) (layers "F.Cu" "F.Paste" "F.Mask") (roundrect_rratio 0.25)
-      (net 1 "GND") (pintype "passive"))
-    (pad "2" smd roundrect (at 0.775 0) (size 0.9 0.95) (layers "F.Cu" "F.Paste" "F.Mask") (roundrect_rratio 0.25)
-      (net 3 "+3V3") (pintype "passive"))
-    (model "${KICAD6_3DMODEL_DIR}/Capacitor_SMD.3dshapes/C_0603_1608Metric.wrl"
-      (offset (xyz 0 0 0))
-      (scale (xyz 1 1 1))
-      (rotate (xyz 0 0 0))
     )
   )
@@
       (offset (xyz 0 0 0))
       (scale (xyz 1 1 1))
+      (rotate (xyz 0 0 0))
+    )
+  )
+  (footprint "Capacitor_SMD:C_0603_1608Metric" (layer "B.Cu")
+    (at 78.255 58.69 180)
+    (descr "Capacitor SMD 0603 (1608 Metric), square (rectangular) end terminal, IPC_7351 nominal, (Body size source: IPC-SM-782 page 76, https://www.pcb-3d.com/wordpress/wp-content/uploads/ipc-sm-782a_amendment_1_and_2.pdf), generated with kicad-footprint-generator")
+    (tags "capacitor")
+    (property "Sheetfile" "miura_board.kicad_sch")
+    (property "Sheetname" "")
+    (attr smd)
+    (fp_text reference "C17" (at 0 1.43) (layer "B.SilkS")
+      (effects (font (size 1 1) (thickness 0.15)) (justify mirror))
+    )
+    (fp_text value "0.1uF" (at 0 -1.43) (layer "B.Fab")
+      (effects (font (size 1 1) (thickness 0.15)) (justify mirror))
+    )
+    (fp_text user "${REFERENCE}" (at 0 0) (layer "B.Fab")
+      (effects (font (size 0.4 0.4) (thickness 0.06)) (justify mirror))
+    )
+    (fp_line (start -0.14058 0.51) (end 0.14058 0.51) (layer "B.SilkS") (width 0.12))
+    (fp_line (start -0.14058 -0.51) (end 0.14058 -0.51) (layer "B.SilkS") (width 0.12))
+    (fp_line (start 1.48 -0.73) (end -1.48 -0.73) (layer "B.CrtYd") (width 0.05))
+    (fp_line (start -1.48 0.73) (end 1.48 0.73) (layer "B.CrtYd") (width 0.05))
+    (fp_line (start 1.48 0.73) (end 1.48 -0.73) (layer "B.CrtYd") (width 0.05))
+    (fp_line (start -1.48 -0.73) (end -1.48 0.73) (layer "B.CrtYd") (width 0.05))
+    (fp_line (start -0.8 -0.4) (end -0.8 0.4) (layer "B.Fab") (width 0.1))
+    (fp_line (start 0.8 0.4) (end 0.8 -0.4) (layer "B.Fab") (width 0.1))
+    (fp_line (start -0.8 0.4) (end 0.8 0.4) (layer "B.Fab") (width 0.1))
+    (fp_line (start 0.8 -0.4) (end -0.8 -0.4) (layer "B.Fab") (width 0.1))
+    (pad "1" smd roundrect (at -0.775 0 180) (size 0.9 0.95) (layers "B.Cu" "B.Paste" "B.Mask") (roundrect_rratio 0.25)
+      (net 1 "GND") (pintype "passive"))
+    (pad "2" smd roundrect (at 0.775 0 180) (size 0.9 0.95) (layers "B.Cu" "B.Paste" "B.Mask") (roundrect_rratio 0.25)
+      (net 3 "+3V3") (pintype "passive"))
+    (model "${KICAD6_3DMODEL_DIR}/Capacitor_SMD.3dshapes/C_0603_1608Metric.wrl"
+      (offset (xyz 0 0 0))
+      (scale (xyz 1 1 1))
